Commit message: add link_4 and joint_4 to arm urdf

File: models/urdf/arm.urdf (robot description, URDF)
Before this commit: robot arm, 5 links, 4 joints
Links:
- added link link_4, mass 0.5; collision cylinder length=0.05 radius=0.05; visual cylinder length=0.1 radius=0.05
Joints:
- added joint joint_4: type revolute, parent link_3, child link_4, origin xyz=0 0 0.45 rpy=0 0 0, axis 0 1 0, limit lower=-1.57 upper=1.57 effort=100 velocity=1.0

Commit message: update joint limits for joint_2 and joint_3

File: models/urdf/arm.urdf (robot description, URDF)
Before this commit: robot arm, 6 links, 5 joints
Joints:
- joint joint_2: limit lower=-3.14 upper=3.14 effort=100 velocity=1.0 -> lower=-1.57 upper=1.57 effort=100 velocity=1.0
- joint joint_3: limit lower=-3.14 upper=3.14 effort=100 velocity=1.0 -> lower=-2.35 upper=2.35 effort=100 velocity=1.0

Commit message: refactor: renamed links and joints in arm urdf

File: models/urdf/arm.urdf (robot description, URDF)
Before this commit: robot arm, 6 links, 5 joints
Links:
- removed link link_1
- removed link link_2
- removed link link_3
- removed link link_4
- added link forearm_link, mass 0.5; collision cylinder length=0.5 radius=0.05; visual cylinder length=0.5 radius=0.05
- added link shoulder_link, mass 0.5; collision cylinder length=0.2 radius=0.1; visual cylinder length=0.2 radius=0.1
- added link upper_arm_link, mass 0.5; collision cylinder length=0.5 radius=0.075; visual cylinder length=0.5 radius=0.075
- added link wrist_link, mass 0.5; collision cylinder length=0.05 radius=0.05; visual cylinder length=0.1 radius=0.05
Joints:
- removed joint joint_1
- removed joint joint_2
- removed joint joint_3
- removed joint joint_4
- added joint joint_1_hip: type revolute, parent base_link, child shoulder_link, origin xyz=0 0 0.1 rpy=0 0 0, axis 0 0 1, limit lower=-3.14 upper=3.14 effort=100 velocity=1.0
- added joint joint_2_shoulder: type revolute, parent shoulder_link, child upper_arm_link, origin xyz=0 -0.175 0.15 rpy=0 0 0, axis 0 1 0, limit lower=-1.57 upper=1.57 effort=100 velocity=1.0
- added joint joint_3_elbow: type revolute, parent upper_arm_link, child forearm_link, origin xyz=0 0.125 0.45 rpy=0 0 0, axis 0 1 0, limit lower=-2.35 upper=2.35 effort=100 velocity=1.0
- added joint joint_4_wrist: type revolute, parent forearm_link, child wrist_link, origin xyz=0 0 0.45 rpy=0 0 0, axis 0 1 0, limit lower=-1.57 upper=1.57 effort=100 velocity=1.0
