Commit message: feat: add roll joint at the end of the arm

File: src/mujoco_arm_sim/models/urdf/arm.urdf (robot description, URDF)
Before this commit: robot arm, 6 links, 5 joints
Links:
- added link roll_link, mass 0.2; collision cylinder length=0.1 radius=0.04; visual cylinder length=0.1 radius=0.04
Joints:
- added joint joint_5_roll: type revolute, parent wrist_link, child roll_link, origin xyz=0 0 0.05 rpy=0 0 0, axis 0 0 1, limit lower=-3.14 upper=3.14 effort=100 velocity=1.0
